File: Z-/Z-.kicad_pcb (KiCad board)
At the start: 4 copper layers, 98 x 98 mm, 140 parts, among them J1 200528-0100, J2 Conn_Coaxial, J3 Conn_Coaxial, J4 200528-0100, J5 Conn_01x02, K1 IM02DGR, Q1 NX3008NBKS, Q10 NX3008NBKS, Q11 IRLML2803, Q12 MBT2222ADW1T1, Q13 IRLML2803, Q14 NX3008NBKS, Q15 IRF7404, Q16 MBT2222ADW1T1, Q17 IRF7404, Q18 IRLML2803, Q19 IRF7404, Q2 NX3008NBKS, Q3 MBT2222ADW1T1, Q4 MBT2222ADW1T1, Q5 NX3008NBKS, Q6 NX3008NBKS, Q7 MBT2222ADW1T1, Q8 MBT2222ADW1T1, Q9 MMBT2222AT, U1 OPT4003DNPRQ1, U2 LTC4316xDD, U3 ADM1176-1ARMZ-R7, U4 NCV891330PD50R2G, U5 DRV8830DRC

Commit message: Stuff idk
Parts:
- removed the G*** at (139.7, 73.7)
Routing:
- net GND: track 11.5 -> 0.00 mm

Commit message: Review fixes
Parts:
- added R69: 0R (DNI), Resistor_SMD:R_0603_1608Metric, B.Cu at (169.5, 85.3)
- added R70: 0R (DNI), Resistor_SMD:R_0603_1608Metric, B.Cu at (169.5, 83.8)
- added R71: 0R, Resistor_SMD:R_0402_1005Metric, F.Cu at (149.2, 65.3)
- added R72: 0R, Resistor_SMD:R_0402_1005Metric, F.Cu at (150.5, 65.3)
- BA1: value ATB2012-50011-T000 -> DXW21HN5011BL
- J2, J3: value Conn_Coaxial -> U.FL
- moved R37 22.6 mm to (136.9, 81.9), turned to 90 degrees
- moved Q9 20.1 mm to (134.4, 81.5), turned to 90 degrees
- moved R11 15.3 mm to (161.9, 92.6), turned to -90 degrees
- moved D3 14.0 mm to (131.4, 82.0), turned to 90 degrees
- moved R6 13.7 mm to (176.3, 90.5), turned to 90 degrees
- moved R7 13.5 mm to (176.3, 92.2), turned to 90 degrees
- moved R9 10.8 mm to (174.8, 90.5), turned to -90 degrees
- moved R8 10.6 mm to (174.8, 92.2), turned to -90 degrees
- moved U5 9.14 mm to (164.9, 91.9), turned to 180 degrees
- moved R56 6.48 mm to (122.6, 90.9), turned to -90 degrees
- moved R13 3.60 mm to (168.1, 90.6), turned to -90 degrees
- moved C8 3.02 mm to (169.1, 93.2), turned to 0 degrees
- moved FL1 2.68 mm to (170.8, 91.4), turned to 0 degrees
- moved J3 2.54 mm to (149.9, 117.9)
- moved K1 0.97 mm to (124.7, 82.0), turned to 90 degrees
Connections:
- net Net-(U1-ADDR) renamed /I2C Devices/ADDR
- J1 pad 10: VBATT -> VBATT_SENSE
- J1 pad 8: VBATT -> VBATT_SENSE
- J1 pad 9: VBATT -> VBATT_SENSE
- R2 pad 2: VBATT -> VBATT_SENSE
- U3 pad 1: VBATT -> VBATT_SENSE
Routing:
- net VBATT: track 169.8 -> 103.8 mm, vias 3 -> 8
- net /I2C Devices/ADDR: track 1.31 -> 34.1 mm, vias 0 -> 2
- net M_FAULT: track 40.2 -> 15.6 mm
- net BURN_RELAY_A: track 33.7 -> 12.5 mm
- net /coil: track 23635.7 -> 23615.9 mm
- net 3.3V: track 98.5 -> 113.8 mm
- net Net-(JP2-Pad2): track 77.7 -> 63.2 mm
- net /I2C Devices/SDAOUT: track 36.2 -> 47.4 mm, vias 2 -> 3
- net SDA_M: track 70.8 -> 60.3 mm
- net +5V: track 16.7 -> 6.49 mm, vias 2 -> 0
- net SCL_M: track 69.4 -> 60.6 mm
- net /I2C Devices/SCLOUT: track 35.0 -> 43.0 mm, vias 2 -> 3
- net VBATT_SENSE: track 0.00 -> 7.61 mm
- net /Burn Wires/VBURN_A_IN: track 99.5 -> 107.1 mm
- net Net-(JP1-Pad2): track 68.7 -> 61.6 mm
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- added copper zone on In1.Cu, net VBATT
- added copper zone on B.Cu, net VBATT_SENSE
Other:
- board text removed: "SUN SENSOR"

Commit message: More review fixes
Routing:
- net /Burn Wires/VBURN_A_IN: track 107.1 -> 7.55 mm
- net VBATT: track 103.8 -> 27.7 mm
- net GND: vias 90 -> 107
Other:
- board text added: "SUN SENSOR"

Commit message: stuff
Parts:
- added Ref**: Val**, custom-footprints:ypanel, F.Cu at (149.4, 54.3)
- AE3: value GPS Antenna -> CGGBP.18.4.A.02
Connections:
- J5 pad MP: (no net) -> GND
Routing:
- net /I2C Devices/ADDR: track 34.1 -> 27.6 mm, vias 2 -> 0
- net Net-(JP1-Pad2): track 61.6 -> 62.6 mm
- net SDA_LS: track 66.3 -> 65.6 mm
Other:
- board text added: "+"
- board text added: "-"
- board text added: "ARGUS-1"
- board text removed: "SUN SENSOR"
